File: kicad/wally.kicad_pcb (KiCad board)
At the start: 4 copper layers, 50 x 30 mm, 36 parts, among them J1 USB C, J2 HDMI_A, J3 HDMI_A, J4 Debug, Q1 AO3401A, Q2 AO3401A, Q3 AO3401A, Q4 AO3400A, SW1 Boot, U1 STM32F042F6Px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

Commit message: Wally v1.01
Parts:
- removed Q2, Q3: AO3401A, Package_TO_SOT_SMD:SOT-23
- removed R13: 10k, Resistor_SMD:R_0603_1608Metric
- removed SW1: Boot, wally:TACT-SWITCH
- added C6: 100n, Capacitor_SMD:C_0402_1005Metric, F.Cu at (153.7, 95.8)
- added C7: 100n, Capacitor_SMD:C_0402_1005Metric, F.Cu at (153.7, 105.7)
- added C8: 100n, Capacitor_SMD:C_0402_1005Metric, F.Cu at (145.9, 95.3)
- added D10: ESD5Z5.0, Diode_SMD:D_SOD-523, F.Cu at (132.8, 103.6)
- added D3: ESD5Z5.0, Diode_SMD:D_SOD-523, F.Cu at (165.6, 101.6)
- added D4: LED, LED_SMD:LED_0402_1005Metric, F.Cu at (168.2, 105.8)
- added D5: ESD5Z5.0, Diode_SMD:D_SOD-523, F.Cu at (173.5, 108.1)
- added D6: LED, LED_SMD:LED_0402_1005Metric, F.Cu at (168.2, 94.2)
- added D7: ESD5Z5.0, Diode_SMD:D_SOD-523, F.Cu at (137.1, 103.6)
- added D8: ESD5Z5.0, Diode_SMD:D_SOD-523, F.Cu at (134.2, 103.6)
- added D9: ESD5Z5.0, Diode_SMD:D_SOD-523, F.Cu at (135.7, 103.6)
- added J5: HDMI Expansion, Connector_PinHeader_1.27mm:PinHeader_1x08_P1.27mm_Vertical, F.Cu at (140.8, 104.4)
- added R18: 1k5, Resistor_SMD:R_0402_1005Metric, F.Cu at (145.9, 104.5)
- added U4: AP2152, Package_SO:MSOP-8_3x3mm_P0.65mm, F.Cu at (150.0, 105.0)
- C1, C2, C3: footprint Capacitor_SMD:C_0603_1608Metric -> Capacitor_SMD:C_0402_1005Metric
- C5: value 1u -> 10u
- D1: value SP0505BAHT -> ESD5Z5.0; footprint Package_TO_SOT_SMD:SOT-23-6 -> Diode_SMD:D_SOD-523
- D2: value LED -> ESD5Z5.0; footprint LED_SMD:LED_0603_1608Metric -> Diode_SMD:D_SOD-523
- J2: footprint wally:AMPHENOL_10029449-001RLF -> Connector_HDMI:HDMI_A_Contact_Technology_HDMI-19APL2_Horizontal; moved to F.Cu
- J3: footprint wally:AMPHENOL_10029449-001RLF -> Connector_HDMI:HDMI_A_Contact_Technology_HDMI-19APL2_Horizontal; moved to B.Cu
- J4: footprint Connector_PinHeader_2.54mm:PinHeader_2x07_P2.54mm_Vertical -> Connector_PinHeader_2.54mm:PinHeader_1x06_P2.54mm_Vertical
- Q1: value AO3401A -> NDC7002N; footprint Package_TO_SOT_SMD:SOT-23 -> Package_TO_SOT_SMD:SuperSOT-6
- R1, R14, R2, R3, R9: footprint Resistor_SMD:R_0603_1608Metric -> Resistor_SMD:R_0402_1005Metric
- R10, R15: value 20k -> 40k; footprint Resistor_SMD:R_0603_1608Metric -> Resistor_SMD:R_0402_1005Metric
- R11, R16: value 30k -> 60k; footprint Resistor_SMD:R_0603_1608Metric -> Resistor_SMD:R_0402_1005Metric
- R12, R8: value 10k -> 1k; footprint Resistor_SMD:R_0603_1608Metric -> Resistor_SMD:R_0402_1005Metric
- R17: value 1k -> 1k5; footprint Resistor_SMD:R_0603_1608Metric -> Resistor_SMD:R_0402_1005Metric
- R4, R5: value 100 -> 20k; footprint Resistor_SMD:R_0603_1608Metric -> Resistor_SMD:R_0402_1005Metric
- R6, R7: value 1k5 -> 100k; footprint Resistor_SMD:R_0603_1608Metric -> Resistor_SMD:R_0402_1005Metric
- U3: value SRV05-4 -> AP2152; footprint Package_TO_SOT_SMD:SOT-23-6 -> Package_SO:MSOP-8_3x3mm_P0.65mm
- moved R12 21.3 mm to (166.3, 94.2)
- moved R8 20.7 mm to (166.3, 105.8)
- moved R16 20.4 mm to (145.9, 92.4), turned to 180 degrees
- moved R17 19.1 mm to (145.9, 105.5)
- moved R15 18.9 mm to (145.9, 93.4), turned to 0 degrees
- moved C4 17.5 mm to (171.8, 108.1), turned to 90 degrees
- moved U2 17.5 mm to (169.1, 108.1)
- moved C5 17.5 mm to (166.3, 108.1)
- moved R9 17.4 mm to (145.9, 94.3), turned to 180 degrees
- moved U3 15.3 mm to (150.0, 95.0), turned to 180 degrees
- moved R14 15.1 mm to (160.0, 106.1), turned to 90 degrees
- moved D2 14.8 mm to (165.6, 98.4), turned to 90 degrees
- moved R3 13.2 mm to (158.0, 95.6), turned to 90 degrees
- moved J4 13.0 mm to (172.2, 91.8)
- moved Q4 12.9 mm to (157.8, 106.1), turned to 180 degrees
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Connections:
- D1 pad 1: hdmi_cec -> hdmi_hpd
- D2 pad 1: Net-(D2-Pad1) -> usb_dp
- D2 pad 2: +3V3 -> GND
- J1 pad S1: Net-(J1-PadS1) -> (no net)
- J4 pad 1: +5V -> GND
- J4 pad 2: +3V3 -> swdio
- J4 pad 3: GND -> swclk
- J4 pad 5: swclk -> uart_rx
- J4 pad 6: swdio -> uart_tx
- Q1 pad 1: hdmi_i2c_en -> +3V3
- Q1 pad 2: hdmi_5v -> i2c_sda
- Q1 pad 3: Net-(Q1-Pad3) -> +3V3
- R12 pad 1: +5V -> Net-(R12-Pad1)
- R12 pad 2: hdmi_5v_en -> Net-(D6-Pad2)
- R17 pad 1: led0 -> Net-(R17-Pad1)
- R17 pad 2: Net-(D2-Pad1) -> hdmi_sda
- R3 pad 1: boot -> hdmi_hpd_en
- R4 pad 1: hdmi_scl -> +3V3
- R5 pad 1: hdmi_sda -> +3V3
- R6 pad 1: Net-(Q1-Pad3) -> +5V
- R7 pad 1: Net-(Q1-Pad3) -> +5V
- R8 pad 1: hdmi_5v -> Net-(R8-Pad1)
- R8 pad 2: hdmi_i2c_en -> Net-(D4-Pad2)
- R9 pad 1: Net-(Q3-Pad3) -> Net-(R9-Pad1)
- U1 pad 1: boot -> hdmi_hpd_en
- U1 pad 10: hdmi_5v_in -> hdmi_5v_en
- U1 pad 12: hdmi_hpd_en -> Net-(R8-Pad1)
- U1 pad 13: hdmi_hpd_in -> Net-(R12-Pad1)
- U1 pad 14: led0 -> (no net)
- U1 pad 6: hdmi_i2c_en -> hdmi_5v_in
- U1 pad 7: hdmi_5v_en -> hdmi_hpd_in
- U3 pad 1: usb_dp -> GND
- U3 pad 2: GND -> +5V
- U3 pad 3: usb_dm -> hdmi_5v_en
- U3 pad 4: usb_dm -> hdmi_hpd_en
- U3 pad 5: +5V -> (no net)
- U3 pad 6: usb_dp -> Net-(R9-Pad1)
Routing:
- net GND: track 98.2 -> 165.8 mm, vias 87 -> 56
- net +5V: track 59.3 -> 86.8 mm, vias 2 -> 3
- net hdmi_5v: track 59.3 -> 32.2 mm
- net boot: track 22.3 -> 0.00 mm, vias 2 -> 0
- net hdmi_hpd_en: track 25.0 -> 7.78 mm
- net Net-(J1-PadS1): track 17.0 -> 0.00 mm
- net hdmi_hpd: track 44.7 -> 28.5 mm
- net hdmi_i2c_en: track 15.4 -> 0.00 mm
- net led0: track 12.3 -> 0.00 mm
- net hdmi_cec_in: track 19.0 -> 7.24 mm
- net Net-(R12-Pad1): track 0.00 -> 11.5 mm, vias 0 -> 2
- net hdmi_5v_in: track 16.6 -> 25.9 mm, vias 2 -> 0
- net i2c_sda: track 19.1 -> 10.3 mm
- net hdmi_cec: track 45.0 -> 52.4 mm
- net hdmi_scl: track 49.3 -> 42.5 mm
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Other:
- board size 50 x 30 mm -> 50 x 20 mm
- board text added: "GND"
- board text added: "RX"
- board text added: "SWCLK"
- board text added: "SWDIO"
- board text added: "TX"
- board text added: "Wally v1.01"
- board text removed: "Wally v1.00"

Commit message: Wally v1.02
Parts:
- C1, C2, C3, C6, C7, C8: footprint Capacitor_SMD:C_0402_1005Metric -> Capacitor_SMD:C_0603_1608Metric
- D4, D6: footprint LED_SMD:LED_0402_1005Metric -> LED_SMD:LED_0603_1608Metric
- J2: moved to B.Cu
- J3: moved to F.Cu
- R1, R10, R11, R12, R14, R15, R16, R17, R18, R2, R3, R4, R5, R6, R7, R8, R9: footprint Resistor_SMD:R_0402_1005Metric -> Resistor_SMD:R_0603_1608Metric
- moved D6 14.4 mm to (162.2, 107.2)
- moved R12 12.3 mm to (162.2, 105.8), turned to 180 degrees
- moved R3 8.77 mm to (150.0, 92.0), turned to 180 degrees
- moved D4 6.69 mm to (162.2, 108.7)
- moved R8 4.41 mm to (162.2, 104.3), turned to 180 degrees
- moved C2 1.88 mm to (157.5, 95.8), turned to 0 degrees
- moved R11 1.55 mm to (145.3, 98.7)
- moved Q4 1.49 mm to (156.4, 105.7)
- moved C1 1.45 mm to (155.2, 99.9)
- moved R14 1.24 mm to (158.9, 105.7)
- moved R16 1.23 mm to (145.3, 91.3)
- moved U1 1.10 mm to (159.8, 100.0)
- moved R10 1.10 mm to (145.3, 97.2)
- moved R6 0.97 mm to (145.3, 102.8)
- moved R7 0.95 mm to (145.3, 107.2)
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Connections:
- R6 pad 1: +5V -> +3V3
- R7 pad 1: +5V -> +3V3
Routing:
- net +5V: track 86.8 -> 72.1 mm
- net +3V3: track 19.0 -> 24.9 mm, vias 7 -> 10
- net Net-(D4-Pad2): track 0.91 -> 6.14 mm
- net Net-(R12-Pad1): track 11.5 -> 6.74 mm, vias 2 -> 0
- net hdmi_hpd_en: track 7.78 -> 12.4 mm, vias 0 -> 2
- net hdmi_sda: track 43.9 -> 46.5 mm, vias 4 -> 3
- net hdmi_scl: track 42.5 -> 40.3 mm
- net Net-(R8-Pad1): track 5.26 -> 3.96 mm
- net i2c_sda: track 10.3 -> 9.22 mm
- net GND: track 165.8 -> 164.7 mm, vias 56 -> 52
- net hdmi_hpd_in: track 25.1 -> 24.1 mm
- net usb_dp: track 7.45 -> 8.46 mm
- net hdmi_5v_in: track 25.9 -> 25.0 mm
- net hdmi_cec_in: track 7.24 -> 6.49 mm
- net uart_tx: track 13.1 -> 12.4 mm
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Other:
- board text added: "Wally v1.02"
- board text removed: "Wally v1.01"

Commit message: v1.02 board bring-up
Parts:
- D10, D8, D9: value ESD5Z5.0 -> ESD5Z3.3
- D4: value LED -> Red LED
- D6: value LED -> Green LED
- Q1: value NDC7002N -> FDC6401N
- R10, R15: value 40k -> 43k
- R11, R16: value 60k -> 62k
- U3, U4: value AP2152 -> STMPS2252

Commit message: Wally v1.03
Parts:
- removed Q1: FDC6401N, Package_TO_SOT_SMD:SuperSOT-6
- removed R6, R7: 100k, Resistor_SMD:R_0603_1608Metric
- added D11: Power LED, LED_SMD:LED_0603_1608Metric, F.Cu at (151.0, 100.0)
- added D12: Yellow LED, LED_SMD:LED_0603_1608Metric, F.Cu at (155.7, 104.3)
- J5: footprint Connector_PinHeader_1.27mm:PinHeader_1x08_P1.27mm_Vertical -> Connector_PinHeader_2.54mm:PinHeader_1x07_P2.54mm_Vertical
- R4, R5: value 20k -> 1k
- moved R5 8.26 mm to (158.7, 104.3), turned to 180 degrees
- moved J5 3.54 mm to (142.4, 107.6)
- moved C6 3.52 mm to (151.0, 97.5), turned to 0 degrees
- moved C7 3.49 mm to (151.0, 107.5), turned to 0 degrees
- moved D1 2.00 mm to (136.5, 103.6)
- moved D10 2.00 mm to (130.8, 103.6)
- moved D7 2.00 mm to (135.1, 103.6)
- moved D8 2.00 mm to (132.2, 103.6)
- moved D9 2.00 mm to (133.7, 103.6)
- moved J2 2.00 mm to (133.0, 108.6)
- moved J3 2.00 mm to (133.0, 91.4)
- moved R4 1.81 mm to (151.0, 101.5), turned to 0 degrees
- moved Q4 1.40 mm to (157.1, 106.9)
- moved R14 1.40 mm to (159.6, 106.9)
- moved U3 1.01 mm to (151.0, 95.0)
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Connections:
- J5 pad 1: +5V -> GND
- J5 pad 2: GND -> hdmi_cec
- J5 pad 3: hdmi_cec -> hdmi_utility
- J5 pad 4: hdmi_utility -> hdmi_scl
- J5 pad 5: hdmi_scl -> hdmi_sda
- J5 pad 6: hdmi_sda -> hdmi_5v
- J5 pad 7: hdmi_5v -> hdmi_hpd
- R4 pad 2: i2c_scl -> Net-(D11-Pad2)
- R5 pad 1: +3V3 -> Net-(R5-Pad1)
- R5 pad 2: i2c_sda -> Net-(D12-Pad2)
- U1 pad 14: (no net) -> Net-(R5-Pad1)
- U1 pad 2: i2c_sda -> hdmi_sda
- U1 pad 3: i2c_scl -> hdmi_scl
Routing:
- net i2c_scl: track 12.9 -> 0.00 mm
- net hdmi_scl: track 40.3 -> 52.6 mm
- net hdmi_sda: track 46.5 -> 55.9 mm
- net i2c_sda: track 9.22 -> 0.00 mm
- net +5V: track 72.1 -> 63.9 mm
- net +3V3: track 24.9 -> 18.3 mm, vias 10 -> 8
- net Net-(R5-Pad1): track 0.00 -> 5.36 mm
- net hdmi_utility: track 25.7 -> 29.7 mm
- net GND: track 164.7 -> 167.8 mm, vias 52 -> 53
- net hdmi_5v: track 32.5 -> 34.7 mm
- net hdmi_hpd: track 28.2 -> 30.2 mm
- net hdmi_5v_en: track 18.4 -> 16.5 mm
- net hdmi_hpd_en: track 12.4 -> 10.8 mm
- net Net-(D11-Pad2): track 0.00 -> 1.52 mm
- net Net-(D12-Pad2): track 0.00 -> 1.38 mm
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Other:
- outline, holes or cut-outs redrawn
- board text added: "Wally v1.03"
- board text removed: "Wally v1.02"

Commit message: Wally v1.04
Parts:
- removed D12: Yellow LED, LED_SMD:LED_0603_1608Metric
- added Q1: FDC6401N, Package_TO_SOT_SMD:SuperSOT-6, F.Cu at (150.4, 100.0)
- added R6: 100k, Resistor_SMD:R_0603_1608Metric, F.Cu at (145.7, 107.2)
- added R7: 100k, Resistor_SMD:R_0603_1608Metric, F.Cu at (145.7, 102.8)
- D11: value Power LED -> ESD5Z5.0; footprint LED_SMD:LED_0603_1608Metric -> Diode_SMD:D_SOD-523
- D8: renamed from D9; value ESD5Z3.3 -> ESD5Z5.0
- D9: renamed from D8; value ESD5Z3.3 -> ESD5Z5.0
- J2, J3: footprint Connector_HDMI:HDMI_A_Contact_Technology_HDMI-19APL2_Horizontal -> wally:HDMI_A_Male_Horizontal
- J4: value Debug -> Expansion; footprint Connector_PinHeader_2.54mm:PinHeader_1x06_P2.54mm_Vertical -> wally:PinHeader_1x09_P2.54mm_Vertical
- R4, R5: value 1k -> 20k
- moved D11 21.9 mm to (129.4, 103.2), turned to 90 degrees
- moved R5 10.7 mm to (150.4, 97.5), turned to 0 degrees
- moved R3 6.47 mm to (156.8, 95.0), turned to 90 degrees
- moved C7 4.17 mm to (154.3, 105.0), turned to 90 degrees
- moved C6 4.17 mm to (154.3, 95.0), turned to 90 degrees
- moved R14 3.38 mm to (157.4, 104.3), turned to 0 degrees
- moved R4 1.15 mm to (150.4, 102.5)
- moved C2 1.11 mm to (158.3, 95.0), turned to 270 degrees
- moved C3 1.09 mm to (161.3, 95.0), turned to 270 degrees
- moved D1 1.07 mm to (161.4, 108.0), turned to 90 degrees
- moved R8 1.06 mm to (162.9, 105.0), turned to 270 degrees
- moved R12 1.05 mm to (161.4, 105.0), turned to 270 degrees
- moved D2 1.05 mm to (162.9, 108.0), turned to 90 degrees
- moved R17 0.62 mm to (145.7, 105.7)
- moved R18 0.62 mm to (145.7, 104.2)
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- renumbered D6 to D1, D4 to D2, D2 to D3, D3 to D4, D1 to D6
Connections:
- D10 pad 1: hdmi_cec -> hdmi_utility
- D11 pad 1: GND -> hdmi_cec
- D11 pad 2: Net-(D11-Pad2) -> GND
- J2 pad SH: GND -> hdmi_sh
- J3 pad SH: GND -> hdmi_sh
- J5 pad 1: GND -> hdmi_cec
- J5 pad 2: hdmi_cec -> hdmi_utility
- J5 pad 3: hdmi_utility -> hdmi_scl
- J5 pad 4: hdmi_scl -> GND
- R17 pad 2: hdmi_sda -> hdmi_scl
- R18 pad 2: hdmi_scl -> hdmi_sda
- R3 pad 1: hdmi_hpd_en -> boot0
- R4 pad 2: Net-(D11-Pad2) -> i2c_scl
- R5 pad 1: Net-(R5-Pad1) -> +3V3
- R5 pad 2: Net-(D12-Pad2) -> i2c_sda
- U1 pad 1: hdmi_hpd_en -> boot0
- U1 pad 10: hdmi_5v_en -> hdmi_hpd_en
- U1 pad 14: Net-(R5-Pad1) -> hdmi_5v_en
- U1 pad 2: hdmi_sda -> i2c_sda
- U1 pad 3: hdmi_scl -> i2c_scl
- U1 pad 6: hdmi_5v_in -> hdmi_hpd_in
- U1 pad 7: hdmi_hpd_in -> hdmi_5v_in
Routing:
- net hdmi_sh: track 0.00 -> 43.1 mm
- net +5V: track 63.9 -> 82.5 mm, vias 3 -> 1
- net Net-(J1-PadSH): track 0.00 -> 17.0 mm
- net GND: track 167.8 -> 182.8 mm, vias 53 -> 55
- net hdmi_5v_in: track 23.8 -> 15.1 mm, vias 0 -> 2
- net i2c_scl: track 0.00 -> 8.58 mm
- net hdmi_utility: track 29.7 -> 37.7 mm
- net i2c_sda: track 0.00 -> 7.51 mm
- net hdmi_5v_en: track 16.5 -> 23.0 mm
- net hdmi_hpd_in: track 23.1 -> 16.7 mm, vias 0 -> 2
- net hdmi_sda: track 55.9 -> 49.6 mm, vias 3 -> 2
- net boot0: track 0.00 -> 6.19 mm
- net Net-(R5-Pad1): track 5.36 -> 0.00 mm
- net hdmi_hpd_en: track 10.8 -> 15.6 mm
- net hdmi_scl: track 52.6 -> 48.2 mm
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Other:
- board text added: "+3.3v"
- board text added: "+5v"
- board text added: "BOOT0"
- board text added: "HDMI +5v"
- board text added: "HDMI CEC"
- board text added: "HDMI HPD"
- board text added: "HDMI SCL"
- board text added: "HDMI SDA"
- board text added: "HDMI UTILITY"
- board text added: "Wally v1.04"
- board text removed: "Wally v1.03"
