File: kicad/wally.sch (KiCad schematic (older format))
At the start: 36 parts, among them J1 USB C, J2 HDMI_A, J3 HDMI_A, J4 Debug, Q1 AO3401A, Q2 AO3401A, Q3 AO3401A, Q4 AO3400A, SW1 Boot, U1 STM32F042F6Px, U2 XC6206PxxxMR, U3 SRV05-4

Commit message: Wally v1.01
Parts:
- removed D1: SP0505BAHT, Package_TO_SOT_SMD:SOT-23-6, symbol Power_Protection:SP0505BAHT
- removed D2: LED, LED_SMD:LED_0603_1608Metric, symbol Device:LED
- removed J1: USB C, wally:USB_C_Receptacle_HRO_TYPE-C-31-M-12, symbol Connector:USB_C_Receptacle_USB2.0
- removed J4: Debug, Connector_PinHeader_2.54mm:PinHeader_2x07_P2.54mm_Vertical, symbol Connector_Generic:Conn_02x07_Odd_Even
- removed Q1, Q2, Q3: AO3401A, Package_TO_SOT_SMD:SOT-23, symbol Transistor_FET:AO3401A
- removed R13: 10k, Resistor_SMD:R_0603_1608Metric, symbol Device:R
- removed SW1: Boot, wally:TACT-SWITCH, symbol Switch:SW_Push
- removed U3: SRV05-4, Package_TO_SOT_SMD:SOT-23-6, symbol Power_Protection:SRV05-4
- added C6, C7, C8: 100n, Capacitor_SMD:C_0402_1005Metric, symbol Device:C
- added D1, D10, D2, D3, D5, D7, D8, D9: ESD5Z5.0, Diode_SMD:D_SOD-523, symbol wally:ESD5Z5.0
- added D4, D6: LED, LED_SMD:LED_0402_1005Metric, symbol Device:LED
- added J1: USB C, wally:USB_C_Receptacle_HRO_TYPE-C-31-M-12, symbol wally:USB_C_Receptacle_USB2.0
- added J4: Debug, Connector_PinHeader_2.54mm:PinHeader_1x06_P2.54mm_Vertical, symbol Connector_Generic:Conn_01x06
- added J5: HDMI Expansion, Connector_PinHeader_1.27mm:PinHeader_1x08_P1.27mm_Vertical, symbol Connector_Generic:Conn_01x08
- added Q1: NDC7002N, Package_TO_SOT_SMD:SuperSOT-6, symbol Device:Q_DUAL_NMOS_G1S2G2D2S1D1
- added R18: 1k5, Resistor_SMD:R_0402_1005Metric, symbol Device:R
- added U3, U4: AP2152, Package_SO:MSOP-8_3x3mm_P0.65mm, symbol wally:AP2152
- C1, C2, C3: footprint Capacitor_SMD:C_0603_1608Metric -> Capacitor_SMD:C_0402_1005Metric
- C5: value 1u -> 10u
- J2, J3: footprint wally:AMPHENOL_10029449-001RLF -> Connector_HDMI:HDMI_A_Contact_Technology_HDMI-19APL2_Horizontal
- R1, R14, R2, R3, R9: footprint Resistor_SMD:R_0603_1608Metric -> Resistor_SMD:R_0402_1005Metric
- R10, R15: value 20k -> 40k; footprint Resistor_SMD:R_0603_1608Metric -> Resistor_SMD:R_0402_1005Metric
- R11, R16: value 30k -> 60k; footprint Resistor_SMD:R_0603_1608Metric -> Resistor_SMD:R_0402_1005Metric
- R12, R8: value 10k -> 1k; footprint Resistor_SMD:R_0603_1608Metric -> Resistor_SMD:R_0402_1005Metric
- R17: value 1k -> 1k5; footprint Resistor_SMD:R_0603_1608Metric -> Resistor_SMD:R_0402_1005Metric
- R4, R5: value 100 -> 20k; footprint Resistor_SMD:R_0603_1608Metric -> Resistor_SMD:R_0402_1005Metric
- R6, R7: value 1k5 -> 100k; footprint Resistor_SMD:R_0603_1608Metric -> Resistor_SMD:R_0402_1005Metric
Connections:
- net boot is gone; now on net hdmi_hpd_en: R3.1, U1.1 (PB8)
- net +3V3: now also R4.1, R5.1, Q1.1 (G), Q1.3 (G)
- net +5V: now also R6.1, R7.1, C6.2, C7.2, D5.1 (A1), J1.A4 (VBUS), J1.A9 (VBUS), J1.B4 (VBUS), J1.B9 (VBUS), J5.1 (Pin_1), U3.2 (IN), U4.2 (IN); no longer R12.1
- net GND: now also C6.1, C7.1, C8.2, D1.2 (A2), D10.2 (A2), D2.2 (A2), D3.2 (A2), D4.1 (K), D5.2 (A2), D6.1 (K), D7.2 (A2), D8.2 (A2), D9.2 (A2), J1.A1 (GND), J1.A12 (GND), J1.B1 (GND), J1.B12 (GND), J4.1 (Pin_1), J4.4 (Pin_4), J5.2 (Pin_2), U3.1 (GND), U4.1 (GND)
- net hdmi_5v: now also C8.1, D7.1 (A1), J5.7 (Pin_7), U3.7 (OUT1); no longer R8.1
- net hdmi_5v_en: now also U1.10 (PA4), U3.3 (EN1), U4.3 (EN1), U4.4 (EN2); no longer R12.2, U1.7 (PA1)
- net hdmi_5v_in: now also U1.6 (PA0); no longer U1.10 (PA4)
- net hdmi_cec: now also D10.1 (A1), J5.3 (Pin_3)
- net hdmi_hpd: now also D1.1 (A1), J5.8 (Pin_8)
- net hdmi_hpd_en: now also U3.4 (EN2); no longer U1.12 (PA6)
- net hdmi_hpd_in: now also U1.7 (PA1); no longer U1.13 (PA7)
- net hdmi_scl: now also D8.1 (A1), J5.5 (Pin_5), Q1.6 (D), R18.2; no longer R4.1
- net hdmi_sda: now also R17.2, D9.1 (A1), J5.6 (Pin_6), Q1.4 (D); no longer R5.1
- net hdmi_utility: now also J5.4 (Pin_4)
- net i2c_scl: now also Q1.5 (S)
- net i2c_sda: now also Q1.2 (S)
- net swclk: now also J4.3 (Pin_3)
- net swdio: now also J4.2 (Pin_2)
- net uart_rx: now also J4.5 (Pin_5)
- net uart_tx: now also J4.6 (Pin_6)
- net usb_dm: now also D3.1 (A1), J1.A7 (D-), J1.B7 (D-)
- net usb_dp: now also D2.1 (A1), J1.A6 (D+), J1.B6 (D+)
- net at R1.2: now also J1.A5 (CC1)
- net at R2.2: now also J1.B5 (CC2)
- net at R9.1: now also U3.6 (OUT2)
- net hdmi_i2c_en: no longer names the net of R8.2
- net hdmi_i2c_en: now also D4.2 (A); no longer U1.6 (PA0)
- net led0: no longer names the net of U1.14 (PB1)
- net led0: no longer R17.1
- new net: R8.1, U1.12 (PA6)
- new net: R12.1, U1.13 (PA7)
- new net: R18.1, U4.6 (OUT2)
- new net: R17.1, U4.7 (OUT1)
- new net: D6.2 (A), R12.2
- no-connect marks 3 -> 8
Other:
- moved on the sheet: C1, C2, C3, C4, C5, Q4, R10, R11, R14, R15, R16, R3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

Commit message: Wally v1.02
Parts:
- C1, C2, C3, C6, C7, C8: footprint Capacitor_SMD:C_0402_1005Metric -> Capacitor_SMD:C_0603_1608Metric
- D4, D6: footprint LED_SMD:LED_0402_1005Metric -> LED_SMD:LED_0603_1608Metric
- R1, R10, R11, R12, R14, R15, R16, R17, R18, R2, R3, R4, R5, R6, R7, R8, R9: footprint Resistor_SMD:R_0402_1005Metric -> Resistor_SMD:R_0603_1608Metric
Connections:
- net +3V3: now also R6.1, R7.1
- net +5V: no longer R6.1, R7.1
Changed lines of the file:
@@
 Sheet 1 1
 Title "Wally"
-Date "2021-04-24"
-Rev "v1.01"
+Date "2021-05-17"
+Rev "v1.02"
 Comp "www.2-0.dk"
 Comment1 ""
@@
 F 0 "R1" V 2700 1850 50  0000 C CNN
 F 1 "5k1" V 2800 1850 50  0000 C CNN
-F 2 "Resistor_SMD:R_0402_1005Metric" V 2730 1850 50  0001 C CNN
+F 2 "Resistor_SMD:R_0603_1608Metric" V 2730 1850 50  0001 C CNN
 F 3 "~" H 2800 1850 50  0001 C CNN
 	1    2800 1850
@@
 F 0 "R2" V 2700 1950 50  0000 C CNN
 F 1 "5k1" V 2800 1950 50  0000 C CNN
-F 2 "Resistor_SMD:R_0402_1005Metric" V 2730 1950 50  0001 C CNN
+F 2 "Resistor_SMD:R_0603_1608Metric" V 2730 1950 50  0001 C CNN
 F 3 "~" H 2800 1950 50  0001 C CNN
 	1    2800 1950
@@
 F 0 "C1" H 4185 5254 50  0000 R CNN
 F 1 "100n" H 4185 5345 50  0000 R CNN
-F 2 "Capacitor_SMD:C_0402_1005Metric" H 4338 5150 50  0001 C CNN
+F 2 "Capacitor_SMD:C_0603_1608Metric" H 4338 5150 50  0001 C CNN
 F 3 "~" H 4300 5300 50  0001 C CNN
 	1    4300 5300
@@
 F 0 "C2" H 4485 4504 50  0000 R CNN
 F 1 "100n" H 4485 4595 50  0000 R CNN
-F 2 "Capacitor_SMD:C_0402_1005Metric" H 4638 4400 50  0001 C CNN
+F 2 "Capacitor_SMD:C_0603_1608Metric" H 4638 4400 50  0001 C CNN
 F 3 "~" H 4600 4550 50  0001 C CNN
 	1    4600 4550
@@
 F 0 "C3" H 4985 4504 50  0000 R CNN
 F 1 "100n" H 4985 4595 50  0000 R CNN
-F 2 "Capacitor_SMD:C_0402_1005Metric" H 5138 4400 50  0001 C CNN
+F 2 "Capacitor_SMD:C_0603_1608Metric" H 5138 4400 50  0001 C CNN
 F 3 "~" H 5100 4550 50  0001 C CNN
 	1    5100 4550
@@
 F 0 "R3" H 4200 6400 50  0000 C CNN
 F 1 "100k" V 4300 6400 50  0000 C CNN
-F 2 "Resistor_SMD:R_0402_1005Metric" V 4230 6400 50  0001 C CNN
+F 2 "Resistor_SMD:R_0603_1608Metric" V 4230 6400 50  0001 C CNN
 F 3 "~" H 4300 6400 50  0001 C CNN
 	1    4300 6400
@@
 F 0 "R14" H 10320 946 50  0000 L CNN
 F 1 "27k" H 10320 855 50  0000 L CNN
-F 2 "Resistor_SMD:R_0402_1005Metric" V 10180 900 50  0001 C CNN
+F 2 "Resistor_SMD:R_0603_1608Metric" V 10180 900 50  0001 C CNN
 F 3 "~" H 10250 900 50  0001 C CNN
 	1    10250 900
@@
 F 0 "R10" H 7870 2546 50  0000 L CNN
 F 1 "40k" H 7870 2455 50  0000 L CNN
-F 2 "Resistor_SMD:R_0402_1005Metric" V 7730 2500 50  0001 C CNN
+F 2 "Resistor_SMD:R_0603_1608Metric" V 7730 2500 50  0001 C CNN
 F 3 "~" H 7800 2500 50  0001 C CNN
 	1    7800 2500
@@
 F 0 "R11" H 7870 2846 50  0000 L CNN
 F 1 "60k" H 7870 2755 50  0000 L CNN
-F 2 "Resistor_SMD:R_0402_1005Metric" V 7730 2800 50  0001 C CNN
+F 2 "Resistor_SMD:R_0603_1608Metric" V 7730 2800 50  0001 C CNN
 F 3 "~" H 7800 2800 50  0001 C CNN
 	1    7800 2800
@@
 F 0 "R15" H 8820 2546 50  0000 L CNN
 F 1 "40k" H 8820 2455 50  0000 L CNN
-F 2 "Resistor_SMD:R_0402_1005Metric" V 8680 2500 50  0001 C CNN
+F 2 "Resistor_SMD:R_0603_1608Metric" V 8680 2500 50  0001 C CNN
 F 3 "~" H 8750 2500 50  0001 C CNN
 	1    8750 2500
@@
 F 0 "R16" H 8820 2846 50  0000 L CNN
 F 1 "60k" H 8820 2755 50  0000 L CNN
-F 2 "Resistor_SMD:R_0402_1005Metric" V 8680 2800 50  0001 C CNN
+F 2 "Resistor_SMD:R_0603_1608Metric" V 8680 2800 50  0001 C CNN
 F 3 "~" H 8750 2800 50  0001 C CNN
 	1    8750 2800
@@
 F 0 "D4" V 6397 6380 50  0000 L CNN
 F 1 "LED" V 6488 6380 50  0000 L CNN
-F 2 "LED_SMD:LED_0402_1005Metric" H 6450 6300 50  0001 C CNN
+F 2 "LED_SMD:LED_0603_1608Metric" H 6450 6300 50  0001 C CNN
 F 3 "~" H 6450 6300 50  0001 C CNN
 	1    6450 6300
@@
 F 0 "R8" H 6520 6046 50  0000 L CNN
 F 1 "1k" H 6520 5955 50  0000 L CNN
-F 2 "Resistor_SMD:R_0402_1005Metric" V 6380 6000 50  0001 C CNN
+F 2 "Resistor_SMD:R_0603_1608Metric" V 6380 6000 50  0001 C CNN
 F 3 "~" H 6450 6000 50  0001 C CNN
 	1    6450 6000
@@
 F 0 "D6" V 6047 6380 50  0000 L CNN
 F 1 "LED" V 6138 6380 50  0000 L CNN
-F 2 "LED_SMD:LED_0402_1005Metric" H 6100 6300 50  0001 C CNN
+F 2 "LED_SMD:LED_0603_1608Metric" H 6100 6300 50  0001 C CNN
 F 3 "~" H 6100 6300 50  0001 C CNN
 	1    6100 6300
@@
 F 0 "R12" H 6170 6046 50  0000 L CNN
 F 1 "1k" H 6170 5955 50  0000 L CNN
-F 2 "Resistor_SMD:R_0402_1005Metric" V 6030 6000 50  0001 C CNN
+F 2 "Resistor_SMD:R_0603_1608Metric" V 6030 6000 50  0001 C CNN
 F 3 "~" H 6100 6000 50  0001 C CNN
 	1    6100 6000
@@
 F 0 "R7" H 9820 3146 50  0000 L CNN
 F 1 "100k" H 9820 3055 50  0000 L CNN
-F 2 "Resistor_SMD:R_0402_1005Metric" V 9680 3100 50  0001 C CNN
+F 2 "Resistor_SMD:R_0603_1608Metric" V 9680 3100 50  0001 C CNN
 F 3 "~" H 9750 3100 50  0001 C CNN
 	1    9750 3100
@@
 F 0 "R6" H 9820 2046 50  0000 L CNN
 F 1 "100k" H 9820 1955 50  0000 L CNN
-F 2 "Resistor_SMD:R_0402_1005Metric" V 9680 2000 50  0001 C CNN
+F 2 "Resistor_SMD:R_0603_1608Metric" V 9680 2000 50  0001 C CNN
 F 3 "~" H 9750 2000 50  0001 C CNN
 	1    9750 2000
@@
 F 0 "R4" H 10320 2046 50  0000 L CNN
 F 1 "20k" H 10320 1955 50  0000 L CNN
-F 2 "Resistor_SMD:R_0402_1005Metric" V 10180 2000 50  0001 C CNN
+F 2 "Resistor_SMD:R_0603_1608Metric" V 10180 2000 50  0001 C CNN
 F 3 "~" H 10250 2000 50  0001 C CNN
 	1    10250 2000
@@
 F 0 "R5" H 10320 3146 50  0000 L CNN
 F 1 "20k" H 10320 3055 50  0000 L CNN
-F 2 "Resistor_SMD:R_0402_1005Metric" V 10180 3100 50  0001 C CNN
+F 2 "Resistor_SMD:R_0603_1608Metric" V 10180 3100 50  0001 C CNN
 F 3 "~" H 10250 3100 50  0001 C CNN
 	1    10250 3100
@@
 F 0 "R9" V 6800 4450 50  0000 C CNN
 F 1 "1k" V 6900 4450 50  0000 C CNN
-F 2 "Resistor_SMD:R_0402_1005Metric" V 6830 4450 50  0001 C CNN
+F 2 "Resistor_SMD:R_0603_1608Metric" V 6830 4450 50  0001 C CNN
 F 3 "~" H 6900 4450 50  0001 C CNN
 	1    6900 4450
@@
 F 0 "C6" V 7250 4950 50  0000 C CNN
 F 1 "100n" V 7350 4950 50  0000 C CNN
-F 2 "Capacitor_SMD:C_0402_1005Metric" H 7538 4800 50  0001 C CNN
+F 2 "Capacitor_SMD:C_0603_1608Metric" H 7538 4800 50  0001 C CNN
 F 3 "~" H 7500 4950 50  0001 C CNN
 	1    7500 4950
@@
 F 0 "C7" V 9750 4950 50  0000 C CNN
 F 1 "100n" V 9850 4950 50  0000 C CNN
-F 2 "Capacitor_SMD:C_0402_1005Metric" H 10038 4800 50  0001 C CNN
+F 2 "Capacitor_SMD:C_0603_1608Metric" H 10038 4800 50  0001 C CNN
 F 3 "~" H 10000 4950 50  0001 C CNN
 	1    10000 4950
@@
 F 0 "R18" V 9500 4450 50  0000 C CNN
 F 1 "1k5" V 9400 4450 50  0000 C CNN
-F 2 "Resistor_SMD:R_0402_1005Metric" V 9330 4450 50  0001 C CNN
+F 2 "Resistor_SMD:R_0603_1608Metric" V 9330 4450 50  0001 C CNN
 F 3 "~" H 9400 4450 50  0001 C CNN
 	1    9400 4450
@@
 F 0 "R17" V 9300 4250 50  0000 C CNN
 F 1 "1k5" V 9400 4250 50  0000 C CNN
-F 2 "Resistor_SMD:R_0402_1005Metric" V 9330 4250 50  0001 C CNN
+F 2 "Resistor_SMD:R_0603_1608Metric" V 9330 4250 50  0001 C CNN
 F 3 "~" H 9400 4250 50  0001 C CNN
 	1    9400 4250
@@
 Wire Wire Line
 	6100 5850 5600 5850
-$Comp
-L power:+5V #PWR050
-U 1 1 60B67268
-P 9750 1850
-F 0 "#PWR050" H 9750 1700 50  0001 C CNN
-F 1 "+5V" H 9765 2023 50  0000 C CNN
-F 2 "" H 9750 1850 50  0001 C CNN
-F 3 "" H 9750 1850 50  0001 C CNN
-	1    9750 1850
-	1    0    0    -1
-$EndComp
-$Comp
-L power:+5V #PWR051
-U 1 1 60B69B9A
-P 9750 2950
-F 0 "#PWR051" H 9750 2800 50  0001 C CNN
-F 1 "+5V" H 9765 3123 50  0000 C CNN
-F 2 "" H 9750 2950 50  0001 C CNN
-F 3 "" H 9750 2950 50  0001 C CNN
-	1    9750 2950
-	1    0    0    -1
-$EndComp
 $Comp
 L power:+5V #PWR04
@@
 F 0 "C8" H 6835 4054 50  0000 R CNN
 F 1 "100n" H 6835 4145 50  0000 R CNN
-F 2 "Capacitor_SMD:C_0402_1005Metric" H 6988 3950 50  0001 C CNN
+F 2 "Capacitor_SMD:C_0603_1608Metric" H 6988 3950 50  0001 C CNN
 F 3 "~" H 6950 4100 50  0001 C CNN
 	1    6950 4100
@@
 $EndComp
 NoConn ~ 1750 3150
+$Comp
+L power:+3.3V #PWR050
+U 1 1 60A32F9D
+P 9750 1850
+F 0 "#PWR050" H 9750 1700 50  0001 C CNN
+F 1 "+3.3V" H 9765 2023 50  0000 C CNN
+F 2 "" H 9750 1850 50  0001 C CNN
+F 3 "" H 9750 1850 50  0001 C CNN
+	1    9750 1850
+	1    0    0    -1
+$EndComp
+$Comp
+L power:+3.3V #PWR051
+U 1 1 60A338EF
+P 9750 2950
+F 0 "#PWR051" H 9750 2800 50  0001 C CNN
+F 1 "+3.3V" H 9765 3123 50  0000 C CNN
+F 2 "" H 9750 2950 50  0001 C CNN
+F 3 "" H 9750 2950 50  0001 C CNN
+	1    9750 2950
+	1    0    0    -1
+$EndComp
 $EndSCHEMATC

Commit message: v1.02 board bring-up
Parts:
- D10, D8, D9: value ESD5Z5.0 -> ESD5Z3.3
- D4: value LED -> Red LED
- D6: value LED -> Green LED
- Q1: value NDC7002N -> FDC6401N
- R10, R15: value 40k -> 43k
- R11, R16: value 60k -> 62k
- U3, U4: value AP2152 -> STMPS2252
Other:
- note added: "5v => 2,95v"
- note added: "5v=> 2,95v"
- note added: "Remove Q1 in next revision."
- moved on the sheet: D4, R8
Changed lines of the file:
@@
 Sheet 1 1
 Title "Wally"
-Date "2021-05-17"
+Date "2021-06-02"
 Rev "v1.02"
 Comp "www.2-0.dk"
@@
 P 7800 2500
 F 0 "R10" H 7870 2546 50  0000 L CNN
-F 1 "40k" H 7870 2455 50  0000 L CNN
+F 1 "43k" H 7870 2455 50  0000 L CNN
 F 2 "Resistor_SMD:R_0603_1608Metric" V 7730 2500 50  0001 C CNN
 F 3 "~" H 7800 2500 50  0001 C CNN
@@
 P 7800 2800
 F 0 "R11" H 7870 2846 50  0000 L CNN
-F 1 "60k" H 7870 2755 50  0000 L CNN
+F 1 "62k" H 7870 2755 50  0000 L CNN
 F 2 "Resistor_SMD:R_0603_1608Metric" V 7730 2800 50  0001 C CNN
 F 3 "~" H 7800 2800 50  0001 C CNN
@@
 P 8750 2500
 F 0 "R15" H 8820 2546 50  0000 L CNN
-F 1 "40k" H 8820 2455 50  0000 L CNN
+F 1 "43k" H 8820 2455 50  0000 L CNN
 F 2 "Resistor_SMD:R_0603_1608Metric" V 8680 2500 50  0001 C CNN
 F 3 "~" H 8750 2500 50  0001 C CNN
@@
 P 8750 2800
 F 0 "R16" H 8820 2846 50  0000 L CNN
-F 1 "60k" H 8820 2755 50  0000 L CNN
+F 1 "62k" H 8820 2755 50  0000 L CNN
 F 2 "Resistor_SMD:R_0603_1608Metric" V 8680 2800 50  0001 C CNN
 F 3 "~" H 8750 2800 50  0001 C CNN
@@
 L Device:LED D4
 U 1 1 608657D3
-P 6450 6300
-F 0 "D4" V 6397 6380 50  0000 L CNN
-F 1 "LED" V 6488 6380 50  0000 L CNN
-F 2 "LED_SMD:LED_0603_1608Metric" H 6450 6300 50  0001 C CNN
-F 3 "~" H 6450 6300 50  0001 C CNN
-	1    6450 6300
+P 6550 6300
+F 0 "D4" V 6497 6380 50  0000 L CNN
+F 1 "Red LED" H 6300 6150 50  0000 L CNN
+F 2 "LED_SMD:LED_0603_1608Metric" H 6550 6300 50  0001 C CNN
+F 3 "~" H 6550 6300 50  0001 C CNN
+	1    6550 6300
 	0    1    -1   0
 $EndComp
@@
 L Device:R R8
 U 1 1 6086A414
-P 6450 6000
-F 0 "R8" H 6520 6046 50  0000 L CNN
-F 1 "1k" H 6520 5955 50  0000 L CNN
-F 2 "Resistor_SMD:R_0603_1608Metric" V 6380 6000 50  0001 C CNN
-F 3 "~" H 6450 6000 50  0001 C CNN
-	1    6450 6000
+P 6550 6000
+F 0 "R8" H 6620 6046 50  0000 L CNN
+F 1 "1k" H 6620 5955 50  0000 L CNN
+F 2 "Resistor_SMD:R_0603_1608Metric" V 6480 6000 50  0001 C CNN
+F 3 "~" H 6550 6000 50  0001 C CNN
+	1    6550 6000
 	1    0    0    -1
 $EndComp
@@
 L power:GND #PWR037
 U 1 1 6086A8A6
-P 6450 6450
-F 0 "#PWR037" H 6450 6200 50  0001 C CNN
-F 1 "GND" H 6455 6277 50  0000 C CNN
-F 2 "" H 6450 6450 50  0001 C CNN
-F 3 "" H 6450 6450 50  0001 C CNN
-	1    6450 6450
+P 6550 6450
+F 0 "#PWR037" H 6550 6200 50  0001 C CNN
+F 1 "GND" H 6555 6277 50  0000 C CNN
+F 2 "" H 6550 6450 50  0001 C CNN
+F 3 "" H 6550 6450 50  0001 C CNN
+	1    6550 6450
 	-1   0    0    -1
 $EndComp
@@
 P 6100 6300
 F 0 "D6" V 6047 6380 50  0000 L CNN
-F 1 "LED" V 6138 6380 50  0000 L CNN
+F 1 "Green LED" H 5850 6150 50  0000 L CNN
 F 2 "LED_SMD:LED_0603_1608Metric" H 6100 6300 50  0001 C CNN
 F 3 "~" H 6100 6300 50  0001 C CNN
@@
 P 8850 5650
 F 0 "D8" H 8800 5550 50  0000 L CNN
-F 1 "ESD5Z5.0" H 8700 5750 50  0000 L CNN
+F 1 "ESD5Z3.3" H 8700 5750 50  0000 L CNN
 F 2 "Diode_SMD:D_SOD-523" H 8850 5450 50  0001 C CNN
 F 3 "" H 8800 5650 50  0001 C CNN
@@
 P 8850 5950
 F 0 "D9" H 8800 5850 50  0000 L CNN
-F 1 "ESD5Z5.0" H 8700 6050 50  0000 L CNN
+F 1 "ESD5Z3.3" H 8700 6050 50  0000 L CNN
 F 2 "Diode_SMD:D_SOD-523" H 8850 5750 50  0001 C CNN
 F 3 "" H 8800 5950 50  0001 C CNN
@@
 P 8850 6250
 F 0 "D10" H 8800 6150 50  0000 L CNN
-F 1 "ESD5Z5.0" H 8700 6350 50  0000 L CNN
+F 1 "ESD5Z3.3" H 8700 6350 50  0000 L CNN
 F 2 "Diode_SMD:D_SOD-523" H 8850 6050 50  0001 C CNN
 F 3 "" H 8800 6250 50  0001 C CNN
@@
 P 7500 4350
 F 0 "U3" H 7500 4915 50  0000 C CNN
-F 1 "AP2152" H 7500 4824 50  0000 C CNN
+F 1 "STMPS2252" H 7500 4824 50  0000 C CNN
 F 2 "Package_SO:MSOP-8_3x3mm_P0.65mm" H 7500 4350 50  0001 C CNN
 F 3 "https://www.diodes.com/assets/Datasheets/AP2142_52.pdf" H 7500 4350 50  0001 C CNN
@@
 P 10000 4350
 F 0 "U4" H 10000 4915 50  0000 C CNN
-F 1 "AP2152" H 10000 4824 50  0000 C CNN
+F 1 "STMPS2252" H 10000 4824 50  0000 C CNN
 F 2 "Package_SO:MSOP-8_3x3mm_P0.65mm" H 10000 4350 50  0001 C CNN
 F 3 "https://www.diodes.com/assets/Datasheets/AP2142_52.pdf" H 10000 4350 50  0001 C CNN
@@
 P 10000 3200
 F 0 "Q1" V 10249 3200 50  0000 C CNN
-F 1 "NDC7002N" V 10340 3200 50  0000 C CNN
+F 1 "FDC6401N" V 10340 3200 50  0000 C CNN
 F 2 "Package_TO_SOT_SMD:SuperSOT-6" H 10200 3200 50  0001 C CNN
 F 3 "~" H 10200 3200 50  0001 C CNN
@@
 P 10000 2100
 F 0 "Q1" V 10249 2100 50  0000 C CNN
-F 1 "NDC7002N" V 10340 2100 50  0000 C CNN
+F 1 "FDC6401N" V 10340 2100 50  0000 C CNN
 F 2 "Package_TO_SOT_SMD:SuperSOT-6" H 10200 2100 50  0001 C CNN
 F 3 "~" H 10200 2100 50  0001 C CNN
@@
 	1    0    0    1
 $EndComp
-Wire Wire Line
-	5600 5750 6450 5750
-Wire Wire Line
-	6450 5750 6450 5850
 NoConn ~ 4400 6150
 Connection ~ 4300 6250
@@
 	1    0    0    -1
 $EndComp
+Text Notes 7900 2600 0    50   ~ 0
+5v => 2,95v
+Text Notes 8850 2600 0    50   ~ 0
+5v=> 2,95v
+Text Notes 9550 2600 0    50   ~ 0
+Remove Q1 in next revision.
+Wire Wire Line
+	5600 5750 6550 5750
+Wire Wire Line
+	6550 5750 6550 5850
 $EndSCHEMATC

Commit message: Wally v1.03
Parts:
- removed J5: HDMI Expansion, Connector_PinHeader_1.27mm:PinHeader_1x08_P1.27mm_Vertical, symbol Connector_Generic:Conn_01x08
- removed Q1: FDC6401N, Package_TO_SOT_SMD:SuperSOT-6, symbol Device:Q_DUAL_NMOS_G1S2G2D2S1D1
- removed R6, R7: 100k, Resistor_SMD:R_0603_1608Metric, symbol Device:R
- added D11: Power LED, LED_SMD:LED_0603_1608Metric, symbol Device:LED
- added D12: Yellow LED, LED_SMD:LED_0603_1608Metric, symbol Device:LED
- added J5: HDMI Expansion, Connector_PinHeader_2.54mm:PinHeader_1x07_P2.54mm_Vertical, symbol Connector_Generic:Conn_01x07
- R4, R5: value 20k -> 1k
Connections:
- net +3V3: no longer R5.1
- net GND: now also D11.1 (K), D12.1 (K), J5.1 (Pin_1)
- net hdmi_5v: now also J5.6 (Pin_6)
- net hdmi_cec: now also J5.2 (Pin_2)
- net hdmi_hpd: now also J5.7 (Pin_7)
- net hdmi_scl: now also U1.3 (PF1), J5.4 (Pin_4)
- net hdmi_sda: now also U1.2 (PF0), J5.5 (Pin_5)
- net hdmi_utility: now also J5.3 (Pin_3)
- net at U1.14 (PB1): now also R5.1
- net i2c_scl: no longer names the net of R4.2
- net i2c_scl: now also D11.2 (A); no longer U1.3 (PF1)
- net i2c_sda: no longer names the net of R5.2
- net i2c_sda: now also D12.2 (A); no longer U1.2 (PF0)
- no-connect marks 8 -> 7
Other:
- note removed: "Remove Q1 in next revision."
- moved on the sheet: Q4, R14

Commit message: Wally v1.04
Parts:
- removed D11: Power LED, LED_SMD:LED_0603_1608Metric, symbol Device:LED
- removed D12: Yellow LED, LED_SMD:LED_0603_1608Metric, symbol Device:LED
- removed J4: Debug, Connector_PinHeader_2.54mm:PinHeader_1x06_P2.54mm_Vertical, symbol Connector_Generic:Conn_01x06
- added D11: ESD5Z5.0, Diode_SMD:D_SOD-523, symbol wally:ESD5Z5.0
- added J4: Expansion, wally:PinHeader_1x09_P2.54mm_Vertical, symbol Connector_Generic:Conn_01x09
- added Q1: FDC6401N, Package_TO_SOT_SMD:SuperSOT-6, symbol Device:Q_DUAL_NMOS_G1S2G2D2S1D1
- added R6, R7: 100k, Resistor_SMD:R_0603_1608Metric, symbol Device:R
- D8: renamed from D9; value ESD5Z3.3 -> ESD5Z5.0
- D9: renamed from D8; value ESD5Z3.3 -> ESD5Z5.0
- J2, J3: footprint Connector_HDMI:HDMI_A_Contact_Technology_HDMI-19APL2_Horizontal -> wally:HDMI_A_Male_Horizontal
- R4, R5: value 1k -> 20k
- renumbered D6 to D1, D4 to D2, D2 to D3, D3 to D4, D1 to D6
Connections:
- net +3V3: now also R5.1, J4.9 (Pin_9), Q1.1 (G), Q1.3 (G)
- net +5V: now also J4.8 (Pin_8), R6.2, R7.2
- net GND: now also J5.4 (Pin_4), D11.2 (A2), J4.1 (Pin_1), J4.4 (Pin_4); no longer J2.SH, J3.SH, J5.1 (Pin_1)
- net hdmi_5v_en: now also U1.14 (PB1); no longer U1.10 (PA4)
- net hdmi_5v_in: now also U1.7 (PA1); no longer U1.6 (PA0)
- net hdmi_cec: now also J5.1 (Pin_1), D11.1 (A1); no longer D10.1 (A1), J5.2 (Pin_2)
- net hdmi_hpd_en: now also U1.10 (PA4); no longer R3.1, U1.1 (PB8)
- net hdmi_hpd_in: now also U1.6 (PA0); no longer U1.7 (PA1)
- net hdmi_scl: now also J5.3 (Pin_3), R17.2, Q1.2 (S), R6.1; no longer J5.4 (Pin_4), R18.2, U1.3 (PF1)
- net hdmi_sda: now also R18.2, Q1.5 (S), R7.1; no longer R17.2, U1.2 (PF0)
- net hdmi_utility: now also D10.1 (A1), J5.2 (Pin_2); no longer J5.3 (Pin_3)
- net swclk: now also J4.3 (Pin_3)
- net swdio: now also J4.2 (Pin_2)
- net uart_rx: now also J4.5 (Pin_5)
- net uart_tx: now also J4.6 (Pin_6)
- net i2c_sda: now reaches R5.2
- net i2c_sda: now also U1.2 (PF0), Q1.6 (D)
- net i2c_scl: now reaches R4.2
- net i2c_scl: now also U1.3 (PF1), Q1.4 (D)
- new net boot0: J4.7 (Pin_7), R3.1, U1.1 (PB8)
- new net hdmi_sh: J2.SH, J3.SH
Other:
- moved on the sheet: D10, D6, D7, D8, D9, Q4, R10, R11, R14, R15, R16, R3
